File: blinken/blinken.kicad_pcb (KiCad board)
At the start: 2 copper layers, 70.7 x 53.5 mm, 50 parts, among them J1 USB_B_Micro, J2 Conn_01x06_Male, J3 Conn_01x02_Male, M1 Fan, M3 Vibrator, Q1 MMBT2222A, Q3 MMBT2222A, SW1 SW_DIP_x10, U1 74HC165, U2 LM1117-3.3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

Commit message: Final revision of pcb
Parts:
- added G***: LOGO, blinken:logo, B.Cu at (110.8, 110.5)
- J2: footprint Connector_PinHeader_2.54mm:PinHeader_1x06_P2.54mm_Vertical -> blinken:programming-pins
- J3, M1, M3: footprint Connector_PinHeader_2.54mm:PinHeader_1x02_P2.54mm_Vertical -> blinken:pads1x2
- U6: footprint Package_SO:SOIC-8_5.275x5.275mm_P1.27mm -> Package_SO:SOIC-8_3.9x4.9mm_P1.27mm
- moved J2 4.15 mm to (118.7, 132.2), turned to 0 degrees
- moved M1 1.34 mm to (144.0, 87.2), turned to -90 degrees
- moved M3 1.32 mm to (144.0, 106.1), turned to -90 degrees
- moved J3 1.23 mm to (144.1, 115.0), turned to -90 degrees
Connections:
- J2 pad 3: /TX -> /RX
- J2 pad 4: /RX -> /TX
Routing:
- net /BOOT: track 27.4 -> 33.1 mm
- net /RX: track 39.8 -> 37.9 mm
- net /TX: track 42.2 -> 44.0 mm
- net /EN: track 48.2 -> 46.5 mm, vias 1 -> 2
- net /CE: track 3.64 -> 4.77 mm
- net /SCK: track 16.7 -> 17.9 mm
- net /SO: track 6.50 -> 7.55 mm
- net GND: track 194.4 -> 195.3 mm, vias 10 -> 11
Other:
- board text added: "flag{d0_y0u_ev3n_t4mp3r_br0}"
