File: blinken/blinken.kicad_sch (KiCad schematic)
At the start: 50 parts, among them J1 USB_B_Micro, J2 Conn_01x06_Male, J3 Conn_01x02_Male, M1 Fan, M3 Vibrator, Q1 MMBT2222A, Q3 MMBT2222A, SW1 SW_DIP_x10, U1 74HC165, U2 LM1117-3.3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

Commit message: Final revision of pcb
Parts:
- J2: footprint Connector_PinHeader_2.54mm:PinHeader_1x06_P2.54mm_Vertical -> blinken:programming-pins
- J3, M1, M3: footprint Connector_PinHeader_2.54mm:PinHeader_1x02_P2.54mm_Vertical -> blinken:pads1x2
- U6: footprint Package_SO:SOIC-8_5.275x5.275mm_P1.27mm -> Package_SO:SOIC-8_3.9x4.9mm_P1.27mm
Connections:
- net RX: now also J2.3 (Pin_3); no longer J2.4 (Pin_4)
- net TX: now also J2.4 (Pin_4); no longer J2.3 (Pin_3)
